File: USBLiPo.sch (EAGLE design)
At the start: 15 parts, among them IC1 LTC4054, J1 USB, Q1 2N7002

Commit message: Layout and overlay
Parts:
- removed J1: USB, freetronics-luke:USB-FT
- added X1: USBSF-MICROB, freetronics-jon:USBSF-MICROB
- B1: value LiPo cell -> 2P-JST-PTH; device freetronics-luke:2P-JST-TH-RA -> freetronics-jon:FREETRONICS-LUKE_2P-JST-TH-RAPTH
Connections:
- net GND: now also B1.NEG, X1.FIX1, X1.FIX2, X1.GND, X1.TAB1, X1.TAB2; no longer B1.-, J1.GND, J1.SH$1
- net N$113: now also X1.VBUS; no longer J1.VBUS
- net N$4: now also B1.POS; no longer B1.+
Other:
- note added: "SMD micro-B USB socket"
- note added: "V1.0 (24-06-2012)"
- note removed: "SMD mini-B USB socket"
- note removed: "V0.5 (08-05-2012)"
- moved on the sheet: Q1
Changed lines of the file:
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@@
 <part name="U$4" library="freetronics-luke" deviceset="GND" device=""/>
 <part name="U$6" library="freetronics-luke" deviceset="GND" device=""/>
-<part name="U$7" library="freetronics-luke" deviceset="GND" device=""/>
 <part name="F1" library="freetronics-luke" deviceset="PTC" device="" value="500mA PTC"/>
 <part name="U$2" library="freetronics-luke" deviceset="GND" device=""/>
@@
 <part name="LED1" library="freetronics-master-v1" deviceset="LED" device="0603" value="Charge"/>
 <part name="LED2" library="freetronics-master-v1" deviceset="LED" device="0603" value="Standby"/>
-<part name="J1" library="freetronics-luke" deviceset="USB-FT" device="" value="USB"/>
 <part name="Q1" library="freetronics-luke" deviceset="2N7002" device=""/>
 <part name="R3" library="freetronics" deviceset="RESISTOR" device="0603" value="3k3"/>
@@
 <part name="S1" library="freetronics-luke" deviceset="SJ" device=""/>
 <part name="S2" library="freetronics-luke" deviceset="SJ" device=""/>
-<part name="B1" library="freetronics-luke" deviceset="2P-JST-TH-RA" device="" value="LiPo cell"/>
+<part name="B1" library="freetronics-jon" deviceset="FREETRONICS-LUKE_2P-JST-TH-RA" device="PTH" value="2P-JST-PTH"/>
+<part name="U$9" library="freetronics-luke" deviceset="GND" device=""/>
+<part name="X1" library="freetronics-jon" deviceset="USBSF" device="-MICROB"/>
 </parts>
 <sheets>
@@
 <plain>
 <text x="7.62" y="20.32" size="3.048" layer="94">USB Li-ion/Li-poly Charger Module</text>
-<text x="38.1" y="14.478" size="1.778" layer="94">V0.5 (08-05-2012)</text>
+<text x="38.1" y="14.478" size="1.778" layer="94">V1.0 (24-06-2012)</text>
 <text x="7.62" y="14.478" size="1.778" layer="94">SKU: USBLIPO</text>
 <text x="7.366" y="9.398" size="1.778" layer="94">(C)2012 Freetronics Pty Ltd: www.freetronics.com</text>
 <text x="7.366" y="6.35" size="1.778" layer="94">Released under the TAPR Open Hardware License: www.tapr.org/ohl</text>
 <text x="68.326" y="14.478" size="1.778" layer="94">www.freetronics.com/usblipo</text>
-<text x="22.86" y="86.36" size="1.27" layer="98">SMD mini-B USB socket</text>
+<text x="22.86" y="91.44" size="1.27" layer="98">SMD micro-B USB socket</text>
 <text x="53.34" y="86.36" size="1.27" layer="98">1812</text>
 <text x="55.88" y="55.88" size="1.27" layer="98">0603</text>
-<text x="129.54" y="58.42" size="1.27" layer="98">2.0mm JST</text>
+<text x="170.18" y="73.66" size="1.27" layer="98">2.0mm JST</text>
 <text x="154.94" y="68.58" size="1.27" layer="98">SOT-23</text>
 <text x="124.46" y="101.6" size="1.27" layer="98">0603</text>
@@
 <text x="137.16" y="83.82" size="1.27" layer="98">Green</text>
 <text x="154.94" y="83.82" size="1.27" layer="98">Yellow</text>
-<wire x1="121.92" y1="73.66" x2="142.24" y2="73.66" width="0.3048" layer="98" style="shortdash"/>
-<wire x1="142.24" y1="73.66" x2="142.24" y2="55.88" width="0.3048" layer="98" style="shortdash"/>
-<wire x1="142.24" y1="55.88" x2="121.92" y2="55.88" width="0.3048" layer="98" style="shortdash"/>
-<wire x1="121.92" y1="55.88" x2="121.92" y2="73.66" width="0.3048" layer="98" style="shortdash"/>
 </plain>
 <instances>
@@
 <instance part="U$4" gate="G$1" x="63.5" y="50.8"/>
 <instance part="U$6" gate="G$1" x="149.86" y="50.8" rot="MR0"/>
-<instance part="U$7" gate="G$1" x="127" y="50.8"/>
 <instance part="F1" gate="G$1" x="53.34" y="81.28" smashed="yes">
 <attribute name="NAME" x="50.038" y="86.36" size="1.27" layer="95"/>
 <attribute name="VALUE" x="50.038" y="83.82" size="1.27" layer="96"/>
 </instance>
-<instance part="U$2" gate="G$1" x="43.18" y="50.8"/>
+<instance part="U$2" gate="G$1" x="45.72" y="50.8"/>
 <instance part="R5" gate="G$1" x="91.44" y="60.96" smashed="yes" rot="MR270">
 <attribute name="NAME" x="93.98" y="60.96" size="1.27" layer="95"/>
@@
 <attribute name="VALUE" x="154.94" y="88.9" size="1.27" layer="96"/>
 </instance>
-<instance part="J1" gate="G$1" x="35.56" y="76.2"/>
-<instance part="Q1" gate="G$1" x="149.86" y="76.2" smashed="yes">
+<instance part="Q1" gate="G$1" x="149.86" y="71.12" smashed="yes">
 <attribute name="NAME" x="154.94" y="73.66" size="1.27" layer="95"/>
 <attribute name="VALUE" x="154.94" y="71.12" size="1.27" layer="96"/>
@@
 <attribute name="NAME" x="83.82" y="71.12" size="1.27" layer="95"/>
 </instance>
-<instance part="B1" gate="G$1" x="127" y="66.04" smashed="yes">
-<attribute name="NAME" x="129.54" y="63.5" size="1.27" layer="95" font="vector"/>
-<attribute name="VALUE" x="129.54" y="60.96" size="1.27" layer="96"/>
-</instance>
+<instance part="B1" gate="G$1" x="170.18" y="78.74"/>
+<instance part="U$9" gate="G$1" x="165.1" y="50.8"/>
+<instance part="X1" gate="G$1" x="35.56" y="76.2" rot="R180"/>
 </instances>
 <busses>
@@
 </segment>
 <segment>
-<wire x1="149.86" y1="71.12" x2="149.86" y2="53.34" width="0.1524" layer="91"/>
+<wire x1="149.86" y1="66.04" x2="149.86" y2="53.34" width="0.1524" layer="91"/>
 <pinref part="U$6" gate="G$1" pin="GND"/>
 <pinref part="Q1" gate="G$1" pin="S"/>
 </segment>
 <segment>
-<wire x1="127" y1="53.34" x2="127" y2="63.5" width="0.1524" layer="91"/>
-<pinref part="U$7" gate="G$1" pin="GND"/>
-<pinref part="B1" gate="G$1" pin="-"/>
-</segment>
-<segment>
-<wire x1="40.64" y1="71.12" x2="43.18" y2="71.12" width="0.1524" layer="91"/>
-<wire x1="43.18" y1="71.12" x2="43.18" y2="63.5" width="0.1524" layer="91"/>
-<wire x1="43.18" y1="63.5" x2="43.18" y2="53.34" width="0.1524" layer="91"/>
-<wire x1="43.18" y1="63.5" x2="30.48" y2="63.5" width="0.1524" layer="91"/>
-<wire x1="30.48" y1="63.5" x2="30.48" y2="66.04" width="0.1524" layer="91"/>
-<junction x="43.18" y="63.5"/>
+<wire x1="40.64" y1="71.12" x2="45.72" y2="71.12" width="0.1524" layer="91"/>
+<wire x1="45.72" y1="71.12" x2="45.72" y2="63.5" width="0.1524" layer="91"/>
+<wire x1="45.72" y1="63.5" x2="45.72" y2="53.34" width="0.1524" layer="91"/>
+<wire x1="45.72" y1="63.5" x2="35.56" y2="63.5" width="0.1524" layer="91"/>
+<wire x1="35.56" y1="63.5" x2="35.56" y2="66.04" width="0.1524" layer="91"/>
+<junction x="45.72" y="63.5"/>
 <pinref part="U$2" gate="G$1" pin="GND"/>
-<pinref part="J1" gate="G$1" pin="GND"/>
-<pinref part="J1" gate="G$1" pin="SH$1"/>
+<pinref part="X1" gate="G$1" pin="TAB2"/>
+<pinref part="X1" gate="G$1" pin="GND"/>
+<pinref part="X1" gate="G$1" pin="TAB1"/>
+<wire x1="35.56" y1="86.36" x2="35.56" y2="88.9" width="0.1524" layer="91"/>
+<wire x1="35.56" y1="88.9" x2="45.72" y2="88.9" width="0.1524" layer="91"/>
+<wire x1="45.72" y1="88.9" x2="45.72" y2="71.12" width="0.1524" layer="91"/>
+<junction x="45.72" y="71.12"/>
+<pinref part="X1" gate="G$1" pin="FIX1"/>
+<wire x1="33.02" y1="86.36" x2="33.02" y2="88.9" width="0.1524" layer="91"/>
+<wire x1="33.02" y1="88.9" x2="35.56" y2="88.9" width="0.1524" layer="91"/>
+<pinref part="X1" gate="G$1" pin="FIX2"/>
+<wire x1="33.02" y1="66.04" x2="33.02" y2="63.5" width="0.1524" layer="91"/>
+<wire x1="33.02" y1="63.5" x2="35.56" y2="63.5" width="0.1524" layer="91"/>
+<junction x="35.56" y="63.5"/>
+<junction x="35.56" y="88.9"/>
 </segment>
 <segment>
@@
 <wire x1="81.28" y1="55.88" x2="81.28" y2="53.34" width="0.1524" layer="91"/>
 </segment>
+<segment>
+<pinref part="B1" gate="G$1" pin="NEG"/>
+<wire x1="167.64" y1="78.74" x2="165.1" y2="78.74" width="0.1524" layer="91"/>
+<wire x1="165.1" y1="78.74" x2="165.1" y2="53.34" width="0.1524" layer="91"/>
+<pinref part="U$9" gate="G$1" pin="GND"/>
+</segment>
 </net>
 <net name="N$1" class="0">
 <segment>
-<wire x1="149.86" y1="86.36" x2="149.86" y2="81.28" width="0.1524" layer="91"/>
+<wire x1="149.86" y1="86.36" x2="149.86" y2="76.2" width="0.1524" layer="91"/>
 <pinref part="LED2" gate="G$1" pin="C"/>
 <pinref part="Q1" gate="G$1" pin="D"/>
@@
 <wire x1="40.64" y1="81.28" x2="48.26" y2="81.28" width="0.1524" layer="91"/>
 <pinref part="F1" gate="G$1" pin="P$1"/>
-<pinref part="J1" gate="G$1" pin="VBUS"/>
+<pinref part="X1" gate="G$1" pin="VBUS"/>
 </segment>
 </net>
@@
 <net name="N$6" class="0">
 <segment>
-<wire x1="144.78" y1="76.2" x2="132.08" y2="76.2" width="0.1524" layer="91"/>
+<wire x1="144.78" y1="71.12" x2="132.08" y2="71.12" width="0.1524" layer="91"/>
+<wire x1="132.08" y1="71.12" x2="132.08" y2="76.2" width="0.1524" layer="91"/>
 <wire x1="132.08" y1="76.2" x2="121.92" y2="76.2" width="0.1524" layer="91"/>
 <wire x1="121.92" y1="99.06" x2="121.92" y2="76.2" width="0.1524" layer="91"/>
@@
 <net name="N$4" class="0">
 <segment>
-<wire x1="119.38" y1="81.28" x2="127" y2="81.28" width="0.1524" layer="91"/>
 <pinref part="IC1" gate="G$1" pin="BAT"/>
-<pinref part="B1" gate="G$1" pin="+"/>
-<wire x1="127" y1="81.28" x2="127" y2="71.12" width="0.1524" layer="91"/>
-</segment>
-</net>
+<pinref part="B1" gate="G$1" pin="POS"/>
+<wire x1="119.38" y1="81.28" x2="167.64" y2="81.28" width="0.1524" layer="91"/>
+</segment>
+</net>

Commit message: Overlay and values
Parts:
- R1, R4, R5: value 10k -> 10K
- R2: value 1k -> 1K
- R3: value 3k3 -> 3K3
Other:
- note added: "100 mA"
- note added: "200 mA"
- note added: "403 mA"
- note added: "503 mA"
- note added: "Charge Current Configuration"
- note added: "Charge current"
- note added: "Closed"
- note added: "Input: 5Vdc 500mA"
- note added: "Open"
- note added: "Output"
- note added: "S1"
- note added: "S2"
- note removed: "0 0 100 mA"
- note removed: "0 1 200 mA"
- note removed: "1 0 403 mA"
- note removed: "1 1 503 mA"
- note removed: "S1 S2 Charge current"
Changed lines of the file:
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@@
 <part name="IC1" library="freetronics-luke" deviceset="LTC4054" device=""/>
 <part name="U$1" library="freetronics-luke" deviceset="GND" device=""/>
-<part name="R2" library="freetronics" deviceset="RESISTOR" device="0603" value="1k"/>
-<part name="R1" library="freetronics" deviceset="RESISTOR" device="0603" value="10k"/>
+<part name="R2" library="freetronics" deviceset="RESISTOR" device="0603" value="1K"/>
+<part name="R1" library="freetronics" deviceset="RESISTOR" device="0603" value="10K"/>
 <part name="C1" library="freetronics" deviceset="CAP" device="0603" value="1uF"/>
 <part name="U$4" library="freetronics-luke" deviceset="GND" device=""/>
@@
 <part name="F1" library="freetronics-luke" deviceset="PTC" device="" value="500mA PTC"/>
 <part name="U$2" library="freetronics-luke" deviceset="GND" device=""/>
-<part name="R5" library="freetronics" deviceset="RESISTOR" device="0603" value="10k"/>
+<part name="R5" library="freetronics" deviceset="RESISTOR" device="0603" value="10K"/>
 <part name="U$3" library="freetronics-luke" deviceset="GND" device=""/>
 <part name="LED1" library="freetronics-master-v1" deviceset="LED" device="0603" value="Charge"/>
 <part name="LED2" library="freetronics-master-v1" deviceset="LED" device="0603" value="Standby"/>
 <part name="Q1" library="freetronics-luke" deviceset="2N7002" device=""/>
-<part name="R3" library="freetronics" deviceset="RESISTOR" device="0603" value="3k3"/>
+<part name="R3" library="freetronics" deviceset="RESISTOR" device="0603" value="3K3"/>
 <part name="U$5" library="freetronics-luke" deviceset="GND" device=""/>
-<part name="R4" library="freetronics" deviceset="RESISTOR" device="0603" value="10k"/>
+<part name="R4" library="freetronics" deviceset="RESISTOR" device="0603" value="10K"/>
 <part name="U$8" library="freetronics-luke" deviceset="GND" device=""/>
 <part name="S1" library="freetronics-luke" deviceset="SJ" device=""/>
@@
 <text x="73.66" y="55.88" size="1.27" layer="98">0603</text>
 <text x="83.82" y="55.88" size="1.27" layer="98">0603</text>
-<text x="139.7" y="33.02" size="1.778" layer="98">S1  S2 Charge current</text>
-<text x="139.7" y="27.94" size="1.778" layer="98">0   0  100 mA</text>
-<text x="139.7" y="22.86" size="1.778" layer="98">0   1  200 mA</text>
-<text x="139.7" y="17.78" size="1.778" layer="98">1   0  403 mA</text>
-<text x="139.7" y="12.7" size="1.778" layer="98">1   1  503 mA</text>
-<wire x1="134.62" y1="38.1" x2="175.26" y2="38.1" width="0.1524" layer="98"/>
-<wire x1="175.26" y1="38.1" x2="175.26" y2="10.16" width="0.1524" layer="98"/>
-<wire x1="175.26" y1="10.16" x2="134.62" y2="10.16" width="0.1524" layer="98"/>
-<wire x1="134.62" y1="10.16" x2="134.62" y2="38.1" width="0.1524" layer="98"/>
+<text x="154.94" y="33.02" size="1.778" layer="98">Charge current</text>
+<text x="129.54" y="27.94" size="1.778" layer="98">Open</text>
+<wire x1="127" y1="35.56" x2="139.7" y2="35.56" width="0.1524" layer="98"/>
+<wire x1="139.7" y1="35.56" x2="152.4" y2="35.56" width="0.1524" layer="98"/>
+<wire x1="152.4" y1="35.56" x2="177.8" y2="35.56" width="0.1524" layer="98"/>
+<wire x1="177.8" y1="35.56" x2="177.8" y2="30.48" width="0.1524" layer="98"/>
+<wire x1="177.8" y1="30.48" x2="177.8" y2="10.16" width="0.1524" layer="98"/>
+<wire x1="177.8" y1="10.16" x2="152.4" y2="10.16" width="0.1524" layer="98"/>
+<wire x1="152.4" y1="10.16" x2="139.7" y2="10.16" width="0.1524" layer="98"/>
+<wire x1="139.7" y1="10.16" x2="127" y2="10.16" width="0.1524" layer="98"/>
+<wire x1="127" y1="10.16" x2="127" y2="30.48" width="0.1524" layer="98"/>
 <text x="137.16" y="83.82" size="1.27" layer="98">Green</text>
 <text x="154.94" y="83.82" size="1.27" layer="98">Yellow</text>
+<text x="160.02" y="27.94" size="1.778" layer="98">100 mA</text>
+<text x="142.24" y="27.94" size="1.778" layer="98">Open</text>
+<text x="142.24" y="22.86" size="1.778" layer="98">Closed</text>
+<text x="129.54" y="22.86" size="1.778" layer="98">Open</text>
+<text x="160.02" y="22.86" size="1.778" layer="98">200 mA</text>
+<text x="129.54" y="17.78" size="1.778" layer="98">Closed</text>
+<text x="142.24" y="17.78" size="1.778" layer="98">Open</text>
+<text x="160.02" y="17.78" size="1.778" layer="98">403 mA</text>
+<text x="129.54" y="12.7" size="1.778" layer="98">Closed</text>
+<text x="142.24" y="12.7" size="1.778" layer="98">Closed</text>
+<text x="160.02" y="12.7" size="1.778" layer="98">503 mA</text>
+<text x="129.54" y="33.02" size="1.778" layer="98">S1</text>
+<text x="142.24" y="33.02" size="1.778" layer="98">S2</text>
+<wire x1="127" y1="30.48" x2="127" y2="35.56" width="0.1524" layer="98"/>
+<wire x1="127" y1="30.48" x2="139.7" y2="30.48" width="0.1524" layer="98"/>
+<wire x1="139.7" y1="30.48" x2="152.4" y2="30.48" width="0.1524" layer="98"/>
+<wire x1="152.4" y1="30.48" x2="177.8" y2="30.48" width="0.1524" layer="98"/>
+<wire x1="139.7" y1="10.16" x2="139.7" y2="30.48" width="0.1524" layer="98"/>
+<wire x1="152.4" y1="10.16" x2="152.4" y2="30.48" width="0.1524" layer="98"/>
+<wire x1="139.7" y1="30.48" x2="139.7" y2="35.56" width="0.1524" layer="98"/>
+<wire x1="152.4" y1="30.48" x2="152.4" y2="35.56" width="0.1524" layer="98"/>
+<text x="127" y="38.1" size="1.778" layer="94" ratio="12">Charge Current Configuration</text>
+<text x="20.32" y="96.52" size="1.778" layer="94" ratio="12">Input: 5Vdc 500mA</text>
+<text x="170.18" y="96.52" size="1.778" layer="94" ratio="12">Output</text>
 </plain>
 <instances>

Commit message: Final changes for v1.0 release
Parts:
- removed B1: 2P-JST-PTH, freetronics-jon:FREETRONICS-LUKE_2P-JST-TH-RAPTH
- removed X1: USBSF-MICROB, freetronics-jon:USBSF-MICROB
- added SJ1, SJ2: SJ, freetronics-luke:SJ
- C1: value 1uF -> 1uF 0603
- F1: value 500mA PTC -> 500mA PTC 1812
- LED1: value Charge -> ORANGE 0603
- LED2: value Standby -> GREEN 0603
- Q1: value 2N7002 -> 2N7002 SOT-23
- R1, R4, R5: value 10K -> 10K 0603
- R2: value 1K -> 1K 0603
- R3: value 3K3 -> 3K3 0603
- S1: value SJ -> USBSF-MICROB; device freetronics-luke:SJ -> freetronics-jon:USBSF-MICROB
- S2: value SJ -> 2P-JST-PTH; device freetronics-luke:SJ -> freetronics-jon:FREETRONICS-LUKE_2P-JST-TH-RAPTH
Connections:
- net GND: now also S1.FIX1, S1.FIX2, S1.GND, S1.TAB1, S1.TAB2, S2.NEG; no longer B1.NEG, X1.FIX1, X1.FIX2, X1.GND, X1.TAB1, X1.TAB2
- net N$113: now also S1.VBUS; no longer X1.VBUS
- net N$3: now also SJ1.2, SJ2.2; no longer S1.2, S2.2
- net N$4: now also S2.POS; no longer B1.POS
- net N$5: now also SJ1.1; no longer S1.1
- net N$7: now also SJ2.1; no longer S2.1
Other:
- note added: "(C)2013 Freetronics Pty Ltd: www.freetronics.com"
- note added: "Charge"
- note added: "SJ1"
- note added: "SJ2"
- note added: "Standby"
- note added: "V1.0 (07-04-2013)"
- note removed: "(C)2012 Freetronics Pty Ltd: www.freetronics.com"
- note removed: "0603"
- note removed: "1812"
- note removed: "Green"
- note removed: "S1"
- note removed: "S2"
- note removed: "SOT-23"
- note removed: "V1.0 (24-06-2012)"
- note removed: "Yellow"
- moved on the sheet: C1, F1, LED1, R2, R3, R4
